File: D32 mk2 iss6 ramboard.kicad_pcb (KiCad board)
At the start: 2 copper layers, 117.5 x 53.3 mm, 34 parts, among them IC1 4116, IC2 4116, IC3 4116, IC36 4116, IC37 4116, IC38 4116, IC39 4116, IC4 4116, IC40 4116, IC41 4116, IC42 4116, IC43 4116, IC5 4116, IC6 4116, IC7 4116, IC8 4116, U1 4164, U10 4164, U11 4164, U12 4164, U13 4164, U14 4164, U15 4164, U16 4164, U2 4164, U3 4164, U4 4164, U5 4164, U6 4164, U7 4164, U8 4164, U9 4164

Commit message: feat: decouple power rail
Parts:
- added C1: 330nF, Capacitor_SMD:C_0603_1608Metric, F.Cu at (97.8, 66.0)
- added C10: 330nF, Capacitor_SMD:C_0603_1608Metric, F.Cu at (110.5, 94.6)
- added C11: 330nF, Capacitor_SMD:C_0603_1608Metric, F.Cu at (123.2, 94.6)
- added C12: 330nF, Capacitor_SMD:C_0603_1608Metric, F.Cu at (135.8, 94.6)
- added C13: 330nF, Capacitor_SMD:C_0603_1608Metric, F.Cu at (148.4, 94.6)
- added C14: 330nF, Capacitor_SMD:C_0603_1608Metric, F.Cu at (161.3, 94.6)
- added C15: 330nF, Capacitor_SMD:C_0603_1608Metric, F.Cu at (174.0, 94.6)
- added C16: 330nF, Capacitor_SMD:C_0603_1608Metric, F.Cu at (199.4, 66.0)
- added C2: 330nF, Capacitor_SMD:C_0603_1608Metric, F.Cu at (110.5, 66.0)
- added C3: 330nF, Capacitor_SMD:C_0603_1608Metric, F.Cu at (123.2, 66.0)
- added C4: 330nF, Capacitor_SMD:C_0603_1608Metric, F.Cu at (135.9, 66.0)
- added C5: 330nF, Capacitor_SMD:C_0603_1608Metric, F.Cu at (148.6, 66.0)
- added C6: 330nF, Capacitor_SMD:C_0603_1608Metric, F.Cu at (161.3, 66.0)
- added C7: 330nF, Capacitor_SMD:C_0603_1608Metric, F.Cu at (174.0, 66.0)
- added C8: 330nF, Capacitor_SMD:C_0603_1608Metric, F.Cu at (186.6, 66.0)
- added C9: 330nF, Capacitor_SMD:C_0603_1608Metric, F.Cu at (97.8, 94.6)
- moved D1 6.35 mm to (116.2, 91.4)
Connections:
- IC1 pad 4: Net-(IC1-Pad4) -> Net-(IC1-Pad15)
- IC2 pad 8: unconnected-(IC2-Pad8) -> +5V
- IC3 pad 8: unconnected-(IC3-Pad8) -> +5V
- IC36 pad 8: unconnected-(IC36-Pad8) -> +5V
- IC37 pad 8: unconnected-(IC37-Pad8) -> +5V
- IC38 pad 8: unconnected-(IC38-Pad8) -> +5V
- IC39 pad 8: unconnected-(IC39-Pad8) -> +5V
- IC4 pad 8: unconnected-(IC4-Pad8) -> +5V
- IC40 pad 8: unconnected-(IC40-Pad8) -> +5V
- IC41 pad 8: unconnected-(IC41-Pad8) -> +5V
- IC42 pad 8: unconnected-(IC42-Pad8) -> +5V
- IC43 pad 16: GND -> unconnected-(IC43-Pad16)
- IC43 pad 8: unconnected-(IC43-Pad8) -> +5V
- IC5 pad 8: unconnected-(IC5-Pad8) -> +5V
- IC6 pad 8: unconnected-(IC6-Pad8) -> +5V
- IC7 pad 8: unconnected-(IC7-Pad8) -> +5V
- IC8 pad 8: unconnected-(IC8-Pad8) -> +5V
- U1 pad 4: Net-(IC1-Pad4) -> Net-(IC1-Pad15)
- U1 pad 8: +5V -> Net-(C1-Pad1)
- U10 pad 8: +5V -> Net-(C10-Pad2)
- U11 pad 8: +5V -> Net-(C11-Pad2)
- U12 pad 8: +5V -> Net-(C12-Pad2)
- U13 pad 8: +5V -> Net-(C13-Pad2)
- U14 pad 8: +5V -> Net-(C14-Pad2)
- U15 pad 8: +5V -> Net-(C15-Pad2)
- U16 pad 8: +5V -> Net-(C16-Pad2)
- U2 pad 4: Net-(IC1-Pad4) -> Net-(IC1-Pad15)
- U2 pad 8: +5V -> Net-(C2-Pad2)
- U3 pad 4: Net-(IC1-Pad4) -> Net-(IC1-Pad15)
- U3 pad 8: +5V -> Net-(C3-Pad2)
- U4 pad 4: Net-(IC1-Pad4) -> Net-(IC1-Pad15)
- U4 pad 8: +5V -> Net-(C4-Pad2)
- U5 pad 4: Net-(IC1-Pad4) -> Net-(IC1-Pad15)
- U5 pad 8: +5V -> Net-(C5-Pad2)
- U6 pad 4: Net-(IC1-Pad4) -> Net-(IC1-Pad15)
- U6 pad 8: +5V -> Net-(C6-Pad2)
- U7 pad 4: Net-(IC1-Pad4) -> Net-(IC1-Pad15)
- U7 pad 8: +5V -> Net-(C7-Pad1)
- U8 pad 4: Net-(IC1-Pad4) -> Net-(IC1-Pad15)
- U8 pad 8: +5V -> Net-(C8-Pad1)
- U9 pad 8: +5V -> Net-(C9-Pad2)
Routing:
- net Net-(IC1-Pad15): track 98.0 -> 196.0 mm
- net Net-(IC1-Pad4): track 98.0 -> 0.00 mm
- net +5V: track 224.2 -> 265.1 mm
- net Net-(D1-Pad2): track 12.1 -> 5.72 mm
- net GND: track 109.5 -> 114.9 mm
- net Net-(C8-Pad1): track 0.00 -> 2.80 mm
- net Net-(C13-Pad2): track 0.00 -> 2.78 mm
- net Net-(C12-Pad2): track 0.00 -> 2.78 mm
- net Net-(C16-Pad2): track 0.00 -> 2.75 mm
- net Net-(C1-Pad1): track 0.00 -> 2.75 mm
- net Net-(C15-Pad2): track 0.00 -> 2.73 mm
- net Net-(C14-Pad2): track 0.00 -> 2.73 mm
- net Net-(C9-Pad2): track 0.00 -> 2.73 mm
- net Net-(C11-Pad2): track 0.00 -> 2.73 mm
- net Net-(C10-Pad2): track 0.00 -> 2.73 mm
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Other:
- board text added: "D32 MkII Issue 6 Memory Repair Board Design by Julian Brown"
- board text added: "Revision 0.1 09/02/2022"
