File: D32 mk2 iss6 ramboard.kicad_sch (KiCad schematic)
At the start: 34 parts, among them IC1 4116, IC2 4116, IC3 4116, IC36 4116, IC37 4116, IC38 4116, IC39 4116, IC4 4116, IC40 4116, IC41 4116, IC42 4116, IC43 4116, IC5 4116, IC6 4116, IC7 4116, IC8 4116, U1 4164, U10 4164, U11 4164, U12 4164, U13 4164, U14 4164, U15 4164, U16 4164, U2 4164, U3 4164, U4 4164, U5 4164, U6 4164, U7 4164, U8 4164, U9 4164

Commit message: feat: decouple power rail
Parts:
- added C1, C10, C11, C12, C13, C14, C15, C16, C2, C3, C4, C5, C6, C7, C8, C9: 330nF, Capacitor_SMD:C_0603_1608Metric, symbol Device:C
Connections:
- net +5V: now also IC2.8 (Vcc), IC3.8 (Vcc), IC36.8 (Vcc), IC37.8 (Vcc), IC38.8 (Vcc), IC39.8 (Vcc), IC4.8 (Vcc), IC40.8 (Vcc), IC41.8 (Vcc), IC42.8 (Vcc), IC43.8 (Vcc), IC5.8 (Vcc), IC6.8 (Vcc), IC7.8 (Vcc), IC8.8 (Vcc), C1.2, C10.1, C11.1, C12.1, C13.1, C14.1, C15.1, C16.1, C2.1, C3.1, C4.1, C5.1, C6.1, C7.2, C8.2, C9.1; no longer U1.8 (Vcc), U10.8 (Vcc), U11.8 (Vcc), U12.8 (Vcc), U13.8 (Vcc), U14.8 (Vcc), U15.8 (Vcc), U16.8 (Vcc), U2.8 (Vcc), U3.8 (Vcc), U4.8 (Vcc), U5.8 (Vcc), U6.8 (Vcc), U7.8 (Vcc), U8.8 (Vcc), U9.8 (Vcc)
- net GND: no longer IC43.16 (Vss)
- net at IC1.15 (|CAS), U1.15 (|CAS), U2.15 (|CAS)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: now also IC1.4 (|RAS), U1.4 (|RAS), U2.4 (|RAS), U3.4 (|RAS), U4.4 (|RAS), U5.4 (|RAS), U6.4 (|RAS), U7.4 (|RAS), U8.4 (|RAS)
- new net: C7.1, U7.8 (Vcc)
- new net: C11.2, U11.8 (Vcc)
- new net: C4.2, U4.8 (Vcc)
- new net: C10.2, U10.8 (Vcc)
- new net: C16.2, U16.8 (Vcc)
- new net: C15.2, U15.8 (Vcc)
- new net: C1.1, U1.8 (Vcc)
- new net: C8.1, U8.8 (Vcc)
- new net: C5.2, U5.8 (Vcc)
- new net: C6.2, U6.8 (Vcc)
- new net: C2.2, U2.8 (Vcc)
- new net: C3.2, U3.8 (Vcc)
- new net: C14.2, U14.8 (Vcc)
- new net: C12.2, U12.8 (Vcc)
- new net: C13.2, U13.8 (Vcc)
- new net: C9.2, U9.8 (Vcc)
Other:
- moved on the sheet: D1, IC1, IC2, IC3, IC36, IC37, IC38, IC39, IC4, IC40, IC41, IC42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
